File: PLC-CIM.kicad_pcb (KiCad board)
At the start: 4 copper layers, 153.5 x 73.7 mm, 128 parts, among them IC1 TLP172AM_TPR,E, IC10 TLV9351IDCKR, IC11 TLV9351IDCKR, IC12 TLV9351IDCKR, IC13 TLP172AM_TPR,E, IC14 TLP172AM_TPR,E, IC15 TLP172AM_TPR,E, IC16 TLP172AM_TPR,E, IC17 TLP172AM_TPR,E, IC18 TLP172AM_TPR,E, IC19 TLV9351IDCKR, IC2 TLP172AM_TPR,E, IC20 TLV9351IDCKR, IC21 TLV9351IDCKR, IC22 TLV9351IDCKR, IC23 TLV9351IDCKR, IC24 TLV9351IDCKR, IC25 TLP172AM_TPR,E, IC26 TLP172AM_TPR,E, IC27 TLP172AM_TPR,E, IC28 TLP172AM_TPR,E, IC29 TLP172AM_TPR,E, IC3 TLP172AM_TPR,E, IC30 TLP172AM_TPR,E, IC31 MAX3221IDBRE4, IC32 TLP172AM_TPR,E, IC33 TLP172AM_TPR,E, IC34 TLP172AM_TPR,E, IC35 TLP172AM_TPR,E, IC36 TLP172AM_TPR,E, IC37 TLP172AM_TPR,E, IC38 TLP172AM_TPR,E, IC39 TLP172AM_TPR,E, IC4 TLP172AM_TPR,E, IC40 TLP172AM_TPR,E, IC41 TLP172AM_TPR,E, IC42 TLP172AM_TPR,E, IC43 TLP172AM_TPR,E, IC44 PCA9555PW,118, IC45 TCAN337DCNR, IC46 PCA9555PW,118, IC47 SN65HVD75DR, IC5 TLP172AM_TPR,E, IC6 TLP172AM_TPR,E, IC7 TLV9351IDCKR, IC8 TLV9351IDCKR, IC9 TLV9351IDCKR, J1 TB001-500-10BE, J10 Conn_02x01, J11 Conn_02x05_Odd_Even, J12 TC0203620000G, J13 750678-1, J14 Conn_02x01, J15 Conn_02x01, J16 Conn_02x01, J17 Conn_02x01, J2 TB001-500-10BE, J3 TB001-500-10BE, J4 TC0203620000G, J5 TC0203620000G, J6 TC0203620000G, J7 TC0203620000G, J8 750678-1, J9 Conn_02x01, U1 ESP32-DEVKITC, U2 AT24CM02-SSHM-B

Commit message: Automate library addition * Added script to automagically extract samacsys libraries and put them in corresponding folders. * Note: Requires zsh
Parts:
- removed J1, J2, J3: TB001-500-10BE, LIB_TB001-500-10BE:SHDR10W100P0X500_1X10_5000X900X1250P
- removed J12, J4, J5, J6, J7: TC0203620000G, TC0203620000G:TC0203620000G
- added IC48: TLP172AM_TPR,E, TLP172AM_TPR_E:SOIC127P700X230-6N, F.Cu at (21.7, 37.2)
- added IC49: TLP172AM_TPR,E, TLP172AM_TPR_E:SOIC127P700X230-6N, F.Cu at (21.7, 42.8)
- added IC50: TLP172AM_TPR,E, TLP172AM_TPR_E:SOIC127P700X230-6N, F.Cu at (21.7, 48.2)
- added IC51: TLP172AM_TPR,E, TLP172AM_TPR_E:SOIC127P700X230-6N, F.Cu at (21.7, 53.8)
- added IC52: TLP172AM_TPR,E, TLP172AM_TPR_E:SOIC127P700X230-6N, F.Cu at (21.7, 59.2)
- added IC53: TLP172AM_TPR,E, TLP172AM_TPR_E:SOIC127P700X230-6N, F.Cu at (21.7, 64.8)
- added IC54: TLP172AM_TPR,E, TLP172AM_TPR_E:SOIC127P700X230-6N, F.Cu at (4.35, 37.2)
- added IC55: TLP172AM_TPR,E, TLP172AM_TPR_E:SOIC127P700X230-6N, F.Cu at (4.35, 42.8)
- added IC56: TLP172AM_TPR,E, TLP172AM_TPR_E:SOIC127P700X230-6N, F.Cu at (4.35, 48.2)
- added IC57: TLP172AM_TPR,E, TLP172AM_TPR_E:SOIC127P700X230-6N, F.Cu at (4.35, 53.8)
- added IC58: TLP172AM_TPR,E, TLP172AM_TPR_E:SOIC127P700X230-6N, F.Cu at (4.35, 59.2)
- added IC59: TLP172AM_TPR,E, TLP172AM_TPR_E:SOIC127P700X230-6N, F.Cu at (4.35, 64.8)
- added IC60: TLP172AM_TPR,E, TLP172AM_TPR_E:SOIC127P700X230-6N, F.Cu at (39.0, 2.25)
- added IC61: TLP172AM_TPR,E, TLP172AM_TPR_E:SOIC127P700X230-6N, F.Cu at (39.0, 7.75)
- added IC62: TLP172AM_TPR,E, TLP172AM_TPR_E:SOIC127P700X230-6N, F.Cu at (39.0, 13.2)
- added IC63: TLP172AM_TPR,E, TLP172AM_TPR_E:SOIC127P700X230-6N, F.Cu at (39.0, 18.8)
- added IC64: TLP172AM_TPR,E, TLP172AM_TPR_E:SOIC127P700X230-6N, F.Cu at (39.0, 24.2)
- added IC65: TLP172AM_TPR,E, TLP172AM_TPR_E:SOIC127P700X230-6N, F.Cu at (39.0, 29.8)
- added IC66: TLP172AM_TPR,E, TLP172AM_TPR_E:SOIC127P700X230-6N, F.Cu at (21.7, 2.25)
- added IC67: TLP172AM_TPR,E, TLP172AM_TPR_E:SOIC127P700X230-6N, F.Cu at (21.7, 7.75)
- added IC68: TLP172AM_TPR,E, TLP172AM_TPR_E:SOIC127P700X230-6N, F.Cu at (21.7, 13.2)
- added IC69: TLP172AM_TPR,E, TLP172AM_TPR_E:SOIC127P700X230-6N, F.Cu at (21.7, 18.8)
- added IC70: TLP172AM_TPR,E, TLP172AM_TPR_E:SOIC127P700X230-6N, F.Cu at (21.7, 24.2)
- added IC71: TLP172AM_TPR,E, TLP172AM_TPR_E:SOIC127P700X230-6N, F.Cu at (21.7, 29.8)
- added IC72: TLP172AM_TPR,E, TLP172AM_TPR_E:SOIC127P700X230-6N, F.Cu at (4.35, 2.25)
- added IC73: TLP172AM_TPR,E, TLP172AM_TPR_E:SOIC127P700X230-6N, F.Cu at (4.35, 7.75)
- added IC74: TLP172AM_TPR,E, TLP172AM_TPR_E:SOIC127P700X230-6N, F.Cu at (4.35, 13.2)
- added IC75: TLP172AM_TPR,E, TLP172AM_TPR_E:SOIC127P700X230-6N, F.Cu at (4.35, 18.8)
- added IC76: TLP172AM_TPR,E, TLP172AM_TPR_E:SOIC127P700X230-6N, F.Cu at (4.35, 24.2)
- added IC77: TLP172AM_TPR,E, TLP172AM_TPR_E:SOIC127P700X230-6N, F.Cu at (4.35, 29.8)
- added R55: CRCW1210267RFKEA, CRCW1210267RFKEA:RESC3225X60N, F.Cu at (29.4, 36.6)
- added R56: CRCW1210267RFKEA, CRCW1210267RFKEA:RESC3225X60N, F.Cu at (29.4, 40.9)
- added R57: CRCW1210267RFKEA, CRCW1210267RFKEA:RESC3225X60N, F.Cu at (29.4, 45.1)
- added R58: CRCW1210267RFKEA, CRCW1210267RFKEA:RESC3225X60N, F.Cu at (29.4, 49.4)
- added R59: CRCW1210267RFKEA, CRCW1210267RFKEA:RESC3225X60N, F.Cu at (29.4, 53.6)
- added R60: CRCW1210267RFKEA, CRCW1210267RFKEA:RESC3225X60N, F.Cu at (29.4, 57.9)
- added R61: CRCW1210267RFKEA, CRCW1210267RFKEA:RESC3225X60N, F.Cu at (12.0, 36.6)
- added R62: CRCW1210267RFKEA, CRCW1210267RFKEA:RESC3225X60N, F.Cu at (12.0, 40.9)
- added R63: CRCW1210267RFKEA, CRCW1210267RFKEA:RESC3225X60N, F.Cu at (12.0, 45.1)
- added R64: CRCW1210267RFKEA, CRCW1210267RFKEA:RESC3225X60N, F.Cu at (12.0, 49.4)
- added R65: CRCW1210267RFKEA, CRCW1210267RFKEA:RESC3225X60N, F.Cu at (12.0, 53.6)
- added R66: CRCW1210267RFKEA, CRCW1210267RFKEA:RESC3225X60N, F.Cu at (12.0, 57.9)
- added R67: CRCW1210267RFKEA, CRCW1210267RFKEA:RESC3225X60N, F.Cu at (46.7, 1.62)
- added R68: CRCW1210267RFKEA, CRCW1210267RFKEA:RESC3225X60N, F.Cu at (46.7, 5.88)
- added R69: CRCW1210267RFKEA, CRCW1210267RFKEA:RESC3225X60N, F.Cu at (46.7, 10.1)
- added R70: CRCW1210267RFKEA, CRCW1210267RFKEA:RESC3225X60N, F.Cu at (46.7, 14.4)
- added R71: CRCW1210267RFKEA, CRCW1210267RFKEA:RESC3225X60N, F.Cu at (46.7, 18.6)
- added R72: CRCW1210267RFKEA, CRCW1210267RFKEA:RESC3225X60N, F.Cu at (46.7, 22.9)
- added R73: CRCW1210267RFKEA, CRCW1210267RFKEA:RESC3225X60N, F.Cu at (29.4, 1.62)
- added R74: CRCW1210267RFKEA, CRCW1210267RFKEA:RESC3225X60N, F.Cu at (29.4, 5.88)
- added R75: CRCW1210267RFKEA, CRCW1210267RFKEA:RESC3225X60N, F.Cu at (29.4, 10.1)
- added R76: CRCW1210267RFKEA, CRCW1210267RFKEA:RESC3225X60N, F.Cu at (29.4, 14.4)
- added R77: CRCW1210267RFKEA, CRCW1210267RFKEA:RESC3225X60N, F.Cu at (29.4, 18.6)
- added R78: CRCW1210267RFKEA, CRCW1210267RFKEA:RESC3225X60N, F.Cu at (29.4, 22.9)
- added R79: CRCW1210267RFKEA, CRCW1210267RFKEA:RESC3225X60N, F.Cu at (12.0, 1.62)
- added R80: CRCW1210267RFKEA, CRCW1210267RFKEA:RESC3225X60N, F.Cu at (12.0, 5.88)
- added R81: CRCW1210267RFKEA, CRCW1210267RFKEA:RESC3225X60N, F.Cu at (12.0, 10.1)
- added R82: CRCW1210267RFKEA, CRCW1210267RFKEA:RESC3225X60N, F.Cu at (12.0, 14.4)
- added R83: CRCW1210267RFKEA, CRCW1210267RFKEA:RESC3225X60N, F.Cu at (12.0, 18.6)
- added R84: CRCW1210267RFKEA, CRCW1210267RFKEA:RESC3225X60N, F.Cu at (12.0, 22.9)
- IC1, IC13, IC14, IC15, IC16, IC17, IC18, IC2, IC25, IC26, IC27, IC28, IC29, IC3, IC30, IC32, IC33, IC34, IC35, IC36, IC37, IC38, IC39, IC4, IC40, IC41, IC42, IC43, IC5, IC6: footprint LIB_TLP172AM_TPR,E:SOIC127P700X230-6N -> TLP172AM_TPR_E:SOIC127P700X230-6N
- IC44, IC46: footprint PCA9555PW,118:SOP65P640X110-24N -> PCA9555PW_118:SOP65P640X110-24N
- moved R1 65.6 mm to (236.2, 72.8)
- moved IC1 56.1 mm to (241.5, 90.2)
- moved R24 46.0 mm to (244.3, 116.2)
- moved IC18 45.3 mm to (247.1, 106.9)
- moved IC14 12.7 mm to (109.1, 100.2)
- moved IC25 12.7 mm to (164.3, 100.2)
- moved IC36 12.7 mm to (180.1, 100.2)
- moved IC37 12.7 mm to (172.2, 100.2)
- moved R38 12.7 mm to (152.5, 98.2)
- moved R39 12.7 mm to (144.7, 98.2)
- moved R41 12.7 mm to (128.8, 98.2)
- moved IC13 12.7 mm to (117.0, 100.2)
- moved IC29 12.7 mm to (132.9, 100.2)
- moved IC30 12.7 mm to (124.8, 100.2)
- moved R19 12.7 mm to (113.0, 98.2)
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Connections:
- IC45 pad 6: Net-(IC45-CANL) -> unconnected-(IC45-CANL-Pad6)
- IC45 pad 7: Net-(IC45-CANH) -> unconnected-(IC45-CANH-Pad7)
Routing:
- net +24V: track 535.2 -> 0.00 mm, vias 37 -> 0
- net +3.3V: track 263.2 -> 0.00 mm, vias 5 -> 0
- net SDA: track 212.6 -> 0.00 mm, vias 1 -> 0
- net GPIO_11: track 201.0 -> 0.00 mm
- net SCL: track 195.0 -> 0.00 mm, vias 1 -> 0
- net GPIO_12: track 188.0 -> 0.00 mm
- net /O Block 1/O_ACT_5: track 161.8 -> 0.00 mm, vias 2 -> 0
- net /O Block 1/O_ACT_4: track 151.9 -> 0.00 mm, vias 2 -> 0
- net /O Block 1/O_ACT_3: track 142.9 -> 0.00 mm, vias 2 -> 0
- net /O Block 4/O_ACT_3: track 141.9 -> 0.00 mm, vias 1 -> 0
- net /O Block 4/O_ACT_4: track 136.3 -> 0.00 mm, vias 1 -> 0
- net CAN_RX: track 136.2 -> 0.00 mm, vias 1 -> 0
- net /O Block 2/O_ACT_2: track 136.0 -> 0.00 mm, vias 4 -> 0
- net CAN_TX: track 135.9 -> 0.00 mm, vias 1 -> 0
- net MCU_IN_2: track 134.4 -> 0.00 mm
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- removed copper zone on B.Cu, net GND
- removed copper zone on F.Cu, net GND
- removed copper zone on In1.Cu, net GND
- removed copper zone on In2.Cu, net GND
