File: PLC-CIM.kicad_pcb (KiCad board)
At the start: 4 copper layers, 153.5 x 73.7 mm, 180 parts, among them IC1 TLP172AM_TPR,E, IC10 TLV9351IDCKR, IC11 TLV9351IDCKR, IC12 TLV9351IDCKR, IC13 TLP172AM_TPR,E, IC14 TLP172AM_TPR,E, IC15 TLP172AM_TPR,E, IC16 TLP172AM_TPR,E, IC17 TLP172AM_TPR,E, IC18 TLP172AM_TPR,E, IC19 TLV9351IDCKR, IC2 TLP172AM_TPR,E, IC20 TLV9351IDCKR, IC21 TLV9351IDCKR, IC22 TLV9351IDCKR, IC23 TLV9351IDCKR, IC24 TLV9351IDCKR, IC25 TLP172AM_TPR,E, IC26 TLP172AM_TPR,E, IC27 TLP172AM_TPR,E, IC28 TLP172AM_TPR,E, IC29 TLP172AM_TPR,E, IC3 TLP172AM_TPR,E, IC30 TLP172AM_TPR,E, IC31 MAX3221IDBRE4, IC32 TLP172AM_TPR,E, IC33 TLP172AM_TPR,E, IC34 TLP172AM_TPR,E, IC35 TLP172AM_TPR,E, IC36 TLP172AM_TPR,E, IC37 TLP172AM_TPR,E, IC38 TLP172AM_TPR,E, IC39 TLP172AM_TPR,E, IC4 TLP172AM_TPR,E, IC40 TLP172AM_TPR,E, IC41 TLP172AM_TPR,E, IC42 TLP172AM_TPR,E, IC43 TLP172AM_TPR,E, IC44 PCA9555PW,118, IC45 TCAN337DCNR, IC46 PCA9555PW,118, IC47 SN65HVD75DR, IC48 TLP172AM_TPR,E, IC49 TLP172AM_TPR,E, IC5 TLP172AM_TPR,E, IC50 TLP172AM_TPR,E, IC51 TLP172AM_TPR,E, IC52 TLP172AM_TPR,E, IC53 TLP172AM_TPR,E, IC54 TLP172AM_TPR,E, IC55 TLP172AM_TPR,E, IC56 TLP172AM_TPR,E, IC57 TLP172AM_TPR,E, IC58 TLP172AM_TPR,E, IC59 TLP172AM_TPR,E, IC6 TLP172AM_TPR,E, IC60 TLP172AM_TPR,E, IC61 TLP172AM_TPR,E, IC62 TLP172AM_TPR,E, IC63 TLP172AM_TPR,E, IC64 TLP172AM_TPR,E, IC65 TLP172AM_TPR,E, IC66 TLP172AM_TPR,E, IC67 TLP172AM_TPR,E, IC68 TLP172AM_TPR,E, IC69 TLP172AM_TPR,E, IC7 TLV9351IDCKR, IC70 TLP172AM_TPR,E, IC71 TLP172AM_TPR,E, IC72 TLP172AM_TPR,E, IC73 TLP172AM_TPR,E, IC74 TLP172AM_TPR,E, IC75 TLP172AM_TPR,E, IC76 TLP172AM_TPR,E, IC77 TLP172AM_TPR,E, IC8 TLV9351IDCKR, IC9 TLV9351IDCKR, J10 Conn_02x01, J11 Conn_02x05_Odd_Even, J13 750678-1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

Commit message: something
Parts:
- removed U1: ESP32-DEVKITC, SnapEDA Library:MODULE_ESP32-DEVKITC
- added IC78: ESP32-WROVER-E-N16R8, ESP32-WROVER-E-N16R8:ESP32WROVEREN16R8, F.Cu at (81.3, 73.8)
- added J1: 1985043, 1985043:1985043, F.Cu at (247.2, 129.2)
- added J2: 1985043, 1985043:1985043, F.Cu at (247.2, 144.3)
- added J3: 1985043, 1985043:1985043, F.Cu at (247.2, 159.4)
Other:
- board text removed: "If you can read this, please replace your ESP32"
