File: PLC-CIM.kicad_sch (KiCad schematic)
At the start: 1 part, among them U1 ESP32-DEVKITC

Commit message: something
Parts:
- removed U1: ESP32-DEVKITC, SnapEDA Library:MODULE_ESP32-DEVKITC, symbol ESP32-DEVKITC:ESP32-DEVKITC
- added IC78: ESP32-WROVER-E-N16R8, ESP32-WROVER-E-N16R8:ESP32WROVEREN16R8, symbol ESP32-WROVER-E-N16R8.kicad_sym:ESP32-WROVER-E-N16R8
Connections:
- net GND: now also IC78.1 (GND_1), IC78.15 (GND_2), IC78.38 (GND_3), IC78.39 (GND_4), IC78.40 (GND_5), IC78.41 (GND_6), IC78.42 (GND_7), IC78.43 (GND_8), IC78.44 (GND_9), IC78.45 (GND_10), IC78.46 (GND_11), IC78.47 (GND_12)
- no-connect marks 10 -> 19
Other:
- removed sheet O Block 5
- sheet IO Terminal ports: added +24v, +5v, GND; removed GPO_13, GPO_14, GPO_15, GPO_16, GPO_17, GPO_18
