File: Blocks/IO_Block_1.kicad_sch (KiCad schematic)
At the start: 24 parts, among them IC1 TLP172AM_TPR,E, IC2 TLP172AM_TPR,E, IC3 TLP172AM_TPR,E, IC4 TLP172AM_TPR,E, IC48 TLP172AM_TPR,E, IC49 TLP172AM_TPR,E, IC5 TLP172AM_TPR,E, IC50 TLP172AM_TPR,E, IC51 TLP172AM_TPR,E, IC52 TLP172AM_TPR,E, IC53 TLP172AM_TPR,E, IC6 TLP172AM_TPR,E

Commit message: Testing documentation
Parts:
- removed IC48, IC49, IC50, IC51, IC52, IC53: TLP172AM_TPR,E, TLP172AM_TPR_E:SOIC127P700X230-6N, symbol TLP172AM_TPR_E:TLP172AM_TPR,E
- removed R55, R56, R57, R58, R59, R60: CRCW1210267RFKEA, CRCW1210267RFKEA:RESC3225X60N, symbol CRCW1210267RFKEA:CRCW1210267RFKEA
Connections:
- no-connect marks 24 -> 12
Other:
- note removed: "SINK CIRCUIT"
