File: v2/PLC-CIM.kicad_pcb (KiCad board)
At the start: 4 copper layers, 153.5 x 73.7 mm, 183 parts, among them IC1 TLP172AM_TPR,E, IC10 TLV9351IDCKR, IC11 TLV9351IDCKR, IC12 TLV9351IDCKR, IC13 TLP172AM_TPR,E, IC14 TLP172AM_TPR,E, IC15 TLP172AM_TPR,E, IC16 TLP172AM_TPR,E, IC17 TLP172AM_TPR,E, IC18 TLP172AM_TPR,E, IC19 TLV9351IDCKR, IC2 TLP172AM_TPR,E, IC20 TLV9351IDCKR, IC21 TLV9351IDCKR, IC22 TLV9351IDCKR, IC23 TLV9351IDCKR, IC24 TLV9351IDCKR, IC25 TLP172AM_TPR,E, IC26 TLP172AM_TPR,E, IC27 TLP172AM_TPR,E, IC28 TLP172AM_TPR,E, IC29 TLP172AM_TPR,E, IC3 TLP172AM_TPR,E, IC30 TLP172AM_TPR,E, IC31 MAX3221IDBRE4, IC32 TLP172AM_TPR,E, IC33 TLP172AM_TPR,E, IC34 TLP172AM_TPR,E, IC35 TLP172AM_TPR,E, IC36 TLP172AM_TPR,E, IC37 TLP172AM_TPR,E, IC38 TLP172AM_TPR,E, IC39 TLP172AM_TPR,E, IC4 TLP172AM_TPR,E, IC40 TLP172AM_TPR,E, IC41 TLP172AM_TPR,E, IC42 TLP172AM_TPR,E, IC43 TLP172AM_TPR,E, IC44 PCA9555PW,118, IC45 TCAN337DCNR, IC46 PCA9555PW,118, IC47 SN65HVD75DR, IC48 TLP172AM_TPR,E, IC49 TLP172AM_TPR,E, IC5 TLP172AM_TPR,E, IC50 TLP172AM_TPR,E, IC51 TLP172AM_TPR,E, IC52 TLP172AM_TPR,E, IC53 TLP172AM_TPR,E, IC54 TLP172AM_TPR,E, IC55 TLP172AM_TPR,E, IC56 TLP172AM_TPR,E, IC57 TLP172AM_TPR,E, IC58 TLP172AM_TPR,E, IC59 TLP172AM_TPR,E, IC6 TLP172AM_TPR,E, IC60 TLP172AM_TPR,E, IC61 TLP172AM_TPR,E, IC62 TLP172AM_TPR,E, IC63 TLP172AM_TPR,E, IC64 TLP172AM_TPR,E, IC65 TLP172AM_TPR,E, IC66 TLP172AM_TPR,E, IC67 TLP172AM_TPR,E, IC68 TLP172AM_TPR,E, IC69 TLP172AM_TPR,E, IC7 TLV9351IDCKR, IC70 TLP172AM_TPR,E, IC71 TLP172AM_TPR,E, IC72 TLP172AM_TPR,E, IC73 TLP172AM_TPR,E, IC74 TLP172AM_TPR,E, IC75 TLP172AM_TPR,E, IC76 TLP172AM_TPR,E, IC77 TLP172AM_TPR,E, IC78 ESP32-WROVER-E-N16R8, IC8 TLV9351IDCKR, IC9 TLV9351IDCKR, J1 1985043, J10 Conn_02x01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

Commit message: Start proper work on V2.1
- Replaced all blocks
- Added input blocks
- Added output blocks
- Added initial CAD placement
- Added initial routing
- General system stability improvements to enhance the user's experience
Parts:
- removed C1, C2, C3, C4: 12103C104KAT2A, 12103C104KAT2A:CAPC3325X94N
- removed IC25, IC26, IC27, IC28, IC29, IC30, IC32, IC33, IC34, IC35, IC36, IC37, IC38, IC39, IC40, IC41, IC42, IC43, IC48, IC49, IC50, IC51, IC52, IC53, IC54, IC55, IC56, IC57, IC58, IC59, IC60, IC61, IC62, IC63, IC64, IC65, IC66, IC67, IC68, IC69, IC70, IC71, IC72, IC73, IC74, IC75, IC76, IC77: TLP172AM_TPR,E, TLP172AM_TPR_E:SOIC127P700X230-6N
- removed IC31: MAX3221IDBRE4, MAX3221IDBRE4:SOP65P780X200-16N
- removed IC44, IC46: PCA9555PW,118, PCA9555PW_118:SOP65P640X110-24N
- removed IC45: TCAN337DCNR, TCAN337DCNR:SOT65P280X145-8N
- removed IC47: SN65HVD75DR, SN65HVD75DR:SOIC127P600X175-8N
- removed IC78: ESP32-WROVER-E-N16R8, ESP32-WROVER-E-N16R8:ESP32WROVEREN16R8
- removed J10, J14, J15, J16, J17, J9: Conn_02x01, Connector_PinHeader_2.54mm:PinHeader_2x01_P2.54mm_Vertical
- removed J11: Conn_02x05_Odd_Even, Connector_PinSocket_2.54mm:PinSocket_2x05_P2.54mm_Vertical
- removed J13, J8: 750678-1, 750678-1:7506781
- removed J3: 1985043, 1985043:1985043
- removed R65, R66, R67, R68, R69, R70, R71, R72, R73, R74, R75, R76, R77, R78, R79, R80, R81, R82, R83, R84: CRCW1210267RFKEA, CRCW1210267RFKEA:RESC3225X60N
- removed U2: AT24CM02-SSHM-B, AT24CM02-SSHM-B:SOIC127P600X175-8N
- added PS1: TMR_6-2410WIR, mod:TMR62410WIR, F.Cu at (178.6, 107.5)
- IC1: value TLP172AM_TPR,E -> ESP32-S3-WROOM-1-N8R8; footprint TLP172AM_TPR_E:SOIC127P700X230-6N -> mod:ESP32S3WROOM1N8R8
- IC10, IC11, IC12, IC7, IC8, IC9: value TLV9351IDCKR -> ITS716GFUMA1; footprint TLV9351IDCKR:SOT65P210X110-5N -> mod:SOIC127P1030X265-20N
- IC13, IC14, IC6: value TLP172AM_TPR,E -> ITS716GFUMA1; footprint TLP172AM_TPR_E:SOIC127P700X230-6N -> mod:SOIC127P1030X265-20N
- IC15, IC16, IC17, IC18: value TLP172AM_TPR,E -> PCA9555PW,118; footprint TLP172AM_TPR_E:SOIC127P700X230-6N -> mod:SOP65P640X110-24N
- IC19: value TLV9351IDCKR -> PCA9555PW,118; footprint TLV9351IDCKR:SOT65P210X110-5N -> mod:SOP65P640X110-24N
- IC2, IC3, IC4, IC5: value TLP172AM_TPR,E -> LM2902KPWR; footprint TLP172AM_TPR_E:SOIC127P700X230-6N -> mod:SOP65P640X120-14N
- IC20, IC21, IC22, IC24: value TLV9351IDCKR -> LM2902KPWR; footprint TLV9351IDCKR:SOT65P210X110-5N -> mod:SOP65P640X120-14N
- IC23: value TLV9351IDCKR -> PIC18F57Q83T-I_PT; footprint TLV9351IDCKR:SOT65P210X110-5N -> mod:QFP50P900X900X120-49N
- J1, J2: value 1985043 -> 39880-0540; footprint 1985043:1985043 -> mod:398800540
- R1, R19, R22, R24, R3, R38, R40, R41, R44, R46, R47, R49, R5, R52, R54, R55, R57, R60, R62, R63: value CRCW1210267RFKEA -> 32.4 kΩ; footprint CRCW1210267RFKEA:RESC3225X60N -> mod:RESC1609X55N
- R10, R12, R26, R28, R29, R8: value RK73B2ETTD152J -> 4.02 kΩ; footprint RK73B2ETTD152J:RESC3226X70N -> mod:RESC1609X55N
- R11, R25, R27, R30, R7, R9: value RK73B2ETTD152J -> 32.4 kΩ; footprint RK73B2ETTD152J:RESC3226X70N -> mod:RESC1609X55N
- R13, R15, R18, R31, R34, R36: value RMCF1210FT10K0 -> 4.02 kΩ; footprint RMCF1210FT10K0:RESC3225X70N -> mod:RESC1609X55N
- R14, R16, R17, R32, R33, R35: value RMCF1210FT10K0 -> 32.4 kΩ; footprint RMCF1210FT10K0:RESC3225X70N -> mod:RESC1609X55N
- R2, R20, R21, R23, R37, R39, R4, R42, R43, R45, R48, R50, R51, R53, R56, R58, R59, R6, R61, R64: value CRCW1210267RFKEA -> 4.02 kΩ; footprint CRCW1210267RFKEA:RESC3225X60N -> mod:RESC1609X55N
- moved J2 165.5 mm to (84.1, 115.9)
- moved IC18 163.3 mm to (86.2, 78.7), turned to -90 degrees
- moved R64 162.5 mm to (166.3, 100.4), turned to 180 degrees
- moved R63 161.0 mm to (163.3, 100.4)
- moved R62 158.9 mm to (159.7, 99.7), turned to -90 degrees
- moved R61 158.0 mm to (157.3, 98.7)
- moved R56 141.1 mm to (157.3, 100.4), turned to 180 degrees
- moved R58 140.8 mm to (157.5, 107.7), turned to 180 degrees
- moved R55 140.2 mm to (154.3, 100.4)
- moved R60 139.8 mm to (159.8, 108.4), turned to 90 degrees
- moved R57 139.8 mm to (154.3, 107.7)
- moved R59 139.7 mm to (157.5, 109.4)
- moved R34 130.5 mm to (94.3, 100.4), turned to 180 degrees
- moved R1 129.9 mm to (109.3, 100.4), turned to 0 degrees
- moved R33 125.8 mm to (91.3, 100.4)
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Connections:
- IC1 pad 1: /O Block 1/O_ACT_6 -> Net-(IC1-GND-Pad1)
- IC1 pad 3: Net-(IC1-CATHODE) -> unconnected-(IC1-EN-Pad3)
- IC1 pad 4: +24V -> /A3
- IC1 pad 5: unconnected-(IC1-NP_2-Pad5) -> /A4
- IC1 pad 6: GPIO_6 -> /A5
- IC10 pad 1: GPIO_5 -> +24V
- IC10 pad 2: GND -> GNDPWR
- IC10 pad 3: Net-(IC10-IN-) -> /Power Stage 5/CH1 Enable
- IC10 pad 4: Net-(IC10-IN-) -> unconnected-(IC10-ST1/2-Pad4)
- IC10 pad 5: +24V -> /Power Stage 5/CH2 Enable
- IC11 pad 1: GPIO_4 -> +24V
- IC11 pad 2: GND -> GNDPWR
- IC11 pad 3: Net-(IC11-IN-) -> /Power Stage 6/CH1 Enable
- IC11 pad 4: Net-(IC11-IN-) -> unconnected-(IC11-ST1/2-Pad4)
- IC11 pad 5: +24V -> /Power Stage 6/CH2 Enable
- IC12 pad 1: GPIO_3 -> +24V
- IC12 pad 2: GND -> GNDPWR
- IC12 pad 3: Net-(IC12-IN-) -> /Power Stage 7/CH1 Enable
- IC12 pad 4: Net-(IC12-IN-) -> unconnected-(IC12-ST1/2-Pad4)
- IC12 pad 5: +24V -> /Power Stage 7/CH2 Enable
- IC13 pad 1: /O Block 2/O_ACT_6 -> +24V
- IC13 pad 2: unconnected-(IC13-NP_1-Pad2) -> GNDPWR
- IC13 pad 3: Net-(IC13-CATHODE) -> /Power Stage 8/CH1 Enable
- IC13 pad 4: +24V -> unconnected-(IC13-ST1/2-Pad4)
- IC13 pad 5: unconnected-(IC13-NP_2-Pad5) -> /Power Stage 8/CH2 Enable
- IC13 pad 6: GPIO_12 -> GNDPWR
- IC14 pad 1: /O Block 2/O_ACT_5 -> +24V
- IC14 pad 2: unconnected-(IC14-NP_1-Pad2) -> GNDPWR
- IC14 pad 3: Net-(IC14-CATHODE) -> /Power Stage 9/CH1 Enable
- IC14 pad 4: +24V -> unconnected-(IC14-ST1/2-Pad4)
- IC14 pad 5: unconnected-(IC14-NP_2-Pad5) -> /Power Stage 9/CH2 Enable
- IC14 pad 6: GPIO_11 -> GNDPWR
- IC15 pad 1: /O Block 2/O_ACT_4 -> unconnected-(IC15-~{INT}-Pad1)
- IC15 pad 3: Net-(IC15-CATHODE) -> unconnected-(IC15-A2-Pad3)
- IC15 pad 4: +24V -> /Power Stage 1/CH1 Enable
- IC15 pad 5: unconnected-(IC15-NP_2-Pad5) -> /Power Stage 1/CH2 Enable
- IC15 pad 6: GPIO_10 -> /Power Stage 1/CH3 Enable
- IC16 pad 1: /O Block 2/O_ACT_3 -> unconnected-(IC16-~{INT}-Pad1)
- IC16 pad 3: Net-(IC16-CATHODE) -> unconnected-(IC16-A2-Pad3)
- IC16 pad 4: +24V -> /Power Stage 3/CH1 Enable
- IC16 pad 5: unconnected-(IC16-NP_2-Pad5) -> /Power Stage 3/CH2 Enable
- IC16 pad 6: GPIO_9 -> /Power Stage 3/CH3 Enable
- IC17 pad 1: /O Block 2/O_ACT_2 -> unconnected-(IC17-~{INT}-Pad1)
- IC17 pad 3: Net-(IC17-CATHODE) -> unconnected-(IC17-A2-Pad3)
- IC17 pad 4: +24V -> /Power Stage 5/CH2 Enable
- IC17 pad 5: unconnected-(IC17-NP_2-Pad5) -> /Power Stage 5/CH1 Enable
- IC17 pad 6: GPIO_8 -> /Power Stage 5/CH3 Enable
- IC18 pad 1: /O Block 2/O_ACT_1 -> unconnected-(IC18-~{INT}-Pad1)
- IC18 pad 3: Net-(IC18-CATHODE) -> unconnected-(IC18-A2-Pad3)
- IC18 pad 4: +24V -> /Power Stage 7/CH2 Enable
- IC18 pad 5: unconnected-(IC18-NP_2-Pad5) -> /Power Stage 7/CH1 Enable
- IC18 pad 6: GPIO_7 -> /Power Stage 7/CH3 Enable
- IC19 pad 1: GPIO_8 -> unconnected-(IC19-~{INT}-Pad1)
- IC19 pad 2: GND -> unconnected-(IC19-A1-Pad2)
- IC19 pad 3: Net-(IC19-IN-) -> unconnected-(IC19-A2-Pad3)
- IC19 pad 4: Net-(IC19-IN-) -> /Power Stage 9/CH2 Enable
- IC19 pad 5: +24V -> /Power Stage 9/CH1 Enable
- IC2 pad 1: /O Block 1/O_ACT_5 -> /Analog Stage 6/L_SIG_1
- IC2 pad 2: unconnected-(IC2-NP_1-Pad2) -> /Analog Stage 6/L_SIG_1
- IC2 pad 3: Net-(IC2-CATHODE) -> Net-(IC2-1IN+)
- IC2 pad 4: +24V -> +3.3V
- IC2 pad 5: unconnected-(IC2-NP_2-Pad5) -> Net-(IC2-2IN+)
- IC2 pad 6: GPIO_5 -> /Analog Stage 6/L_SIG_2
- IC20 pad 1: GPIO_7 -> /Analog Stage 5/L_SIG_1
- IC20 pad 2: GND -> /Analog Stage 5/L_SIG_1
- IC20 pad 3: Net-(IC20-IN-) -> Net-(IC20-1IN+)
- IC20 pad 4: Net-(IC20-IN-) -> +3.3V
- IC20 pad 5: +24V -> Net-(IC20-2IN+)
- IC21 pad 1: GPIO_12 -> /Analog Stage 7/L_SIG_1
- IC21 pad 2: GND -> /Analog Stage 7/L_SIG_1
- IC21 pad 3: Net-(IC21-IN-) -> Net-(IC21-1IN+)
- IC21 pad 4: Net-(IC21-IN-) -> +3.3V
- IC21 pad 5: +24V -> Net-(IC21-2IN+)
- IC22 pad 1: GPIO_11 -> /Analog Stage 8/L_SIG_1
- IC22 pad 2: GND -> /Analog Stage 8/L_SIG_1
- IC22 pad 3: Net-(IC22-IN-) -> Net-(IC22-1IN+)
- IC22 pad 4: Net-(IC22-IN-) -> +3.3V
- IC22 pad 5: +24V -> Net-(IC22-2IN+)
- IC23 pad 1: GPIO_10 -> unconnected-(IC23-RC7-Pad1)
- IC23 pad 2: GND -> unconnected-(IC23-RD4-Pad2)
- IC23 pad 3: Net-(IC23-IN-) -> unconnected-(IC23-RD5-Pad3)
- IC23 pad 4: Net-(IC23-IN-) -> unconnected-(IC23-RD6-Pad4)
- IC23 pad 5: +24V -> unconnected-(IC23-RD7-Pad5)
- IC24 pad 1: GPIO_9 -> /A0
- IC24 pad 2: GND -> /A0
- IC24 pad 3: Net-(IC24-IN-) -> Net-(IC24-1IN+)
- IC24 pad 4: Net-(IC24-IN-) -> +3.3V
- IC24 pad 5: +24V -> Net-(IC24-2IN+)
- IC3 pad 1: /O Block 1/O_ACT_4 -> /A4
- IC3 pad 2: unconnected-(IC3-NP_1-Pad2) -> /A4
- IC3 pad 3: Net-(IC3-CATHODE) -> Net-(IC3-1IN+)
- IC3 pad 4: +24V -> +3.3V
- IC3 pad 5: unconnected-(IC3-NP_2-Pad5) -> Net-(IC3-2IN+)
- IC3 pad 6: GPIO_4 -> /A5
- IC4 pad 1: /O Block 1/O_ACT_3 -> /A8
- IC4 pad 2: unconnected-(IC4-NP_1-Pad2) -> /A8
- IC4 pad 3: Net-(IC4-CATHODE) -> Net-(IC4-1IN+)
- IC4 pad 4: +24V -> +3.3V
- IC4 pad 5: unconnected-(IC4-NP_2-Pad5) -> Net-(IC4-2IN+)
- IC4 pad 6: GPIO_3 -> /A9
- IC5 pad 1: /O Block 1/O_ACT_2 -> /A12
- IC5 pad 2: unconnected-(IC5-NP_1-Pad2) -> /A12
- IC5 pad 3: Net-(IC5-CATHODE) -> Net-(IC5-1IN+)
- IC5 pad 4: +24V -> +3.3V
- IC5 pad 5: unconnected-(IC5-NP_2-Pad5) -> Net-(IC5-2IN+)
- IC5 pad 6: GPIO_2 -> /A13
- IC6 pad 1: /O Block 1/O_ACT_1 -> +24V
- IC6 pad 2: unconnected-(IC6-NP_1-Pad2) -> GNDPWR
- IC6 pad 3: Net-(IC6-CATHODE) -> /Power Stage 1/CH1 Enable
- IC6 pad 4: +24V -> unconnected-(IC6-ST1/2-Pad4)
- IC6 pad 5: unconnected-(IC6-NP_2-Pad5) -> /Power Stage 1/CH2 Enable
- IC6 pad 6: GPIO_1 -> GNDPWR
- IC7 pad 1: GPIO_2 -> +24V
- IC7 pad 2: GND -> GNDPWR
- IC7 pad 3: Net-(IC7-IN-) -> /Power Stage 2/CH1 Enable
- IC7 pad 4: Net-(IC7-IN-) -> unconnected-(IC7-ST1/2-Pad4)
- IC7 pad 5: +24V -> /Power Stage 2/CH2 Enable
- IC8 pad 1: GPIO_1 -> +24V
- IC8 pad 2: GND -> GNDPWR
- IC8 pad 3: Net-(IC8-IN-) -> /Power Stage 3/CH1 Enable
- IC8 pad 4: Net-(IC8-IN-) -> unconnected-(IC8-ST1/2-Pad4)
- IC8 pad 5: +24V -> /Power Stage 3/CH2 Enable
- IC9 pad 1: GPIO_6 -> +24V
- IC9 pad 2: GND -> GNDPWR
- IC9 pad 3: Net-(IC9-IN-) -> /Power Stage 4/CH1 Enable
- IC9 pad 4: Net-(IC9-IN-) -> unconnected-(IC9-ST1/2-Pad4)
- IC9 pad 5: +24V -> /Power Stage 4/CH2 Enable
- J1 pad 1: GPIO_1 -> /Power Stage 1/CH1
- J1 pad 10: GPIO_10 -> /Power Stage 3/CH2
- J1 pad 2: GPIO_2 -> /Power Stage 1/CH2
- J1 pad 3: GPIO_3 -> /Power Stage 1/CH3
- J1 pad 4: GPIO_4 -> /Power Stage 1/CH4
- J1 pad 5: GPIO_5 -> /Power Stage 2/CH1
- J1 pad 6: GPIO_6 -> /Power Stage 2/CH2
- J1 pad 7: GPIO_7 -> /Power Stage 2/CH3
- J1 pad 8: GPIO_8 -> /Power Stage 2/CH4
- J1 pad 9: GPIO_9 -> /Power Stage 3/CH1
- J2 pad 1: GPIO_11 -> /Analog Stage 1/H_SIG_1
- J2 pad 10: OUT_20 -> /Analog Stage 3/H_SIG_2
- J2 pad 2: GPIO_12 -> /Analog Stage 1/H_SIG_2
- J2 pad 3: OUT_13 -> /Analog Stage 1/H_SIG_3
- J2 pad 4: OUT_14 -> /Analog Stage 1/H_SIG_4
- J2 pad 5: OUT_15 -> /Analog Stage 2/H_SIG_1
- J2 pad 6: OUT_16 -> /Analog Stage 2/H_SIG_2
- J2 pad 7: OUT_17 -> /Analog Stage 2/H_SIG_3
- J2 pad 8: OUT_18 -> /Analog Stage 2/H_SIG_4
- J2 pad 9: OUT_19 -> /Analog Stage 3/H_SIG_1
- R1 pad 1: Net-(IC1-CATHODE) -> /D4
- R1 pad 2: GND -> Net-(IC2-1IN+)
- R10 pad 1: MCU_IN_8 -> GNDS
- R10 pad 2: GND -> Net-(IC3-1IN+)
- R11 pad 1: MCU_IN_9 -> /Analog Stage 2/H_SIG_2
- R11 pad 2: GND -> Net-(IC3-2IN+)
- R12 pad 1: MCU_IN_10 -> GNDS
- R12 pad 2: GND -> Net-(IC3-2IN+)
- R13 pad 1: Net-(IC7-IN-) -> GNDS
- R13 pad 2: MCU_IN_11 -> Net-(IC3-3IN+)
- R14 pad 1: Net-(IC8-IN-) -> /Analog Stage 2/H_SIG_3
- R14 pad 2: MCU_IN_12 -> Net-(IC3-3IN+)
- R15 pad 1: Net-(IC9-IN-) -> GNDS
- R15 pad 2: MCU_IN_7 -> Net-(IC3-4IN+)
- R16 pad 1: Net-(IC10-IN-) -> /Analog Stage 2/H_SIG_4
- R16 pad 2: MCU_IN_8 -> Net-(IC3-4IN+)
- R17 pad 1: Net-(IC11-IN-) -> /Analog Stage 3/H_SIG_1
- R17 pad 2: MCU_IN_9 -> Net-(IC4-1IN+)
- R18 pad 1: Net-(IC12-IN-) -> GNDS
- R18 pad 2: MCU_IN_10 -> Net-(IC4-1IN+)
- R19 pad 1: Net-(IC13-CATHODE) -> /Analog Stage 3/H_SIG_2
- R19 pad 2: GND -> Net-(IC4-2IN+)
- R2 pad 1: Net-(IC2-CATHODE) -> GNDS
- R2 pad 2: GND -> Net-(IC2-1IN+)
- R20 pad 1: Net-(IC14-CATHODE) -> GNDS
- R20 pad 2: GND -> Net-(IC4-2IN+)
- R21 pad 1: Net-(IC15-CATHODE) -> GNDS
- R21 pad 2: GND -> Net-(IC4-3IN+)
- R22 pad 1: Net-(IC16-CATHODE) -> /Analog Stage 3/H_SIG_3
- R22 pad 2: GND -> Net-(IC4-3IN+)
- R23 pad 1: Net-(IC17-CATHODE) -> GNDS
- R23 pad 2: GND -> Net-(IC4-4IN+)
- R24 pad 1: Net-(IC18-CATHODE) -> /Analog Stage 3/H_SIG_4
- R24 pad 2: GND -> Net-(IC4-4IN+)
- R25 pad 1: MCU_IN_5 -> /Analog Stage 1/H_SIG_1
- R25 pad 2: GND -> Net-(IC24-1IN+)
- R26 pad 1: MCU_IN_6 -> GNDS
- R26 pad 2: GND -> Net-(IC24-1IN+)
- R27 pad 1: MCU_IN_1 -> /Analog Stage 4/H_SIG_2
- R27 pad 2: GND -> Net-(IC5-2IN+)
- R28 pad 1: MCU_IN_2 -> GNDS
- R28 pad 2: GND -> Net-(IC5-2IN+)
- R29 pad 1: MCU_IN_3 -> GNDS
- R29 pad 2: GND -> Net-(IC5-3IN+)
- R3 pad 1: Net-(IC3-CATHODE) -> /Analog Stage 1/H_SIG_2
- R3 pad 2: GND -> Net-(IC24-2IN+)
- R30 pad 1: MCU_IN_4 -> /Analog Stage 4/H_SIG_3
- R30 pad 2: GND -> Net-(IC5-3IN+)
- R31 pad 1: Net-(IC19-IN-) -> GNDS
- R31 pad 2: MCU_IN_5 -> Net-(IC5-4IN+)
- R32 pad 1: Net-(IC20-IN-) -> /Analog Stage 4/H_SIG_4
- R32 pad 2: MCU_IN_6 -> Net-(IC5-4IN+)
- R33 pad 1: Net-(IC21-IN-) -> /D0
- R33 pad 2: MCU_IN_1 -> Net-(IC20-1IN+)
- R34 pad 1: Net-(IC22-IN-) -> GNDS
- R34 pad 2: MCU_IN_2 -> Net-(IC20-1IN+)
- R35 pad 1: Net-(IC23-IN-) -> /D1
- R35 pad 2: MCU_IN_3 -> Net-(IC20-2IN+)
- R36 pad 1: Net-(IC24-IN-) -> GNDS
- R36 pad 2: MCU_IN_4 -> Net-(IC20-2IN+)
- R37 pad 1: Net-(IC25-CATHODE) -> GNDS
- R37 pad 2: GND -> Net-(IC20-3IN+)
- R38 pad 1: Net-(IC26-CATHODE) -> /D2
- R38 pad 2: GND -> Net-(IC20-3IN+)
- R39 pad 1: Net-(IC27-CATHODE) -> GNDS
- R39 pad 2: GND -> Net-(IC20-4IN+)
- R4 pad 1: Net-(IC4-CATHODE) -> GNDS
- R4 pad 2: GND -> Net-(IC24-2IN+)
- R40 pad 1: Net-(IC28-CATHODE) -> /D3
- R40 pad 2: GND -> Net-(IC20-4IN+)
- R41 pad 1: Net-(IC29-CATHODE) -> /D5
- R41 pad 2: GND -> Net-(IC2-2IN+)
- R42 pad 1: Net-(IC30-CATHODE) -> GNDS
- R42 pad 2: GND -> Net-(IC2-2IN+)
- R43 pad 1: Net-(IC32-CATHODE) -> GNDS
- R43 pad 2: GND -> Net-(IC2-3IN+)
- R44 pad 1: Net-(IC33-CATHODE) -> /D6
- R44 pad 2: GND -> Net-(IC2-3IN+)
- R45 pad 1: Net-(IC34-CATHODE) -> GNDS
- R45 pad 2: GND -> Net-(IC2-4IN+)
- R46 pad 1: Net-(IC35-CATHODE) -> /D7
- R46 pad 2: GND -> Net-(IC2-4IN+)
- R47 pad 1: Net-(IC36-CATHODE) -> /D8
- R47 pad 2: GND -> Net-(IC21-1IN+)
- R48 pad 1: Net-(IC37-CATHODE) -> GNDS
- R48 pad 2: GND -> Net-(IC21-1IN+)
- R49 pad 1: Net-(IC38-CATHODE) -> /D9
- R49 pad 2: GND -> Net-(IC21-2IN+)
- R5 pad 1: Net-(IC5-CATHODE) -> /Analog Stage 1/H_SIG_4
- R5 pad 2: GND -> Net-(IC24-4IN+)
- R50 pad 1: Net-(IC39-CATHODE) -> GNDS
- R50 pad 2: GND -> Net-(IC21-2IN+)
- R51 pad 1: Net-(IC40-CATHODE) -> GNDS
- R51 pad 2: GND -> Net-(IC21-3IN+)
- R52 pad 1: Net-(IC41-CATHODE) -> /D10
- R52 pad 2: GND -> Net-(IC21-3IN+)
- R53 pad 1: Net-(IC42-CATHODE) -> GNDS
- R53 pad 2: GND -> Net-(IC21-4IN+)
- R54 pad 1: Net-(IC43-CATHODE) -> /D11
- R54 pad 2: GND -> Net-(IC21-4IN+)
- R55 pad 1: Net-(IC48-CATHODE) -> /D12
- R55 pad 2: GND -> Net-(IC22-1IN+)
- R56 pad 1: Net-(IC49-CATHODE) -> GNDS
- R56 pad 2: GND -> Net-(IC22-1IN+)
- R57 pad 1: Net-(IC50-CATHODE) -> /D13
- R57 pad 2: GND -> Net-(IC22-2IN+)
- R58 pad 1: Net-(IC51-CATHODE) -> GNDS
- R58 pad 2: GND -> Net-(IC22-2IN+)
- R59 pad 1: Net-(IC52-CATHODE) -> GNDS
- R59 pad 2: GND -> Net-(IC22-3IN+)
- R6 pad 1: Net-(IC6-CATHODE) -> GNDS
- R6 pad 2: GND -> Net-(IC24-4IN+)
- R60 pad 1: Net-(IC53-CATHODE) -> /D14
- R60 pad 2: GND -> Net-(IC22-3IN+)
- R61 pad 1: Net-(IC54-CATHODE) -> GNDS
- R61 pad 2: GND -> Net-(IC22-4IN+)
- R62 pad 1: Net-(IC55-CATHODE) -> /D15
- R62 pad 2: GND -> Net-(IC22-4IN+)
- R63 pad 1: Net-(IC56-CATHODE) -> /Analog Stage 4/H_SIG_1
- R63 pad 2: GND -> Net-(IC5-1IN+)
- R64 pad 1: Net-(IC57-CATHODE) -> GNDS
- R64 pad 2: GND -> Net-(IC5-1IN+)
- R7 pad 1: MCU_IN_11 -> /Analog Stage 1/H_SIG_3
- R7 pad 2: GND -> Net-(IC24-3IN+)
- R8 pad 1: MCU_IN_12 -> GNDS
- R8 pad 2: GND -> Net-(IC24-3IN+)
- R9 pad 1: MCU_IN_7 -> /Analog Stage 2/H_SIG_1
- R9 pad 2: GND -> Net-(IC3-1IN+)
Routing:
- net Net-(IC24-3IN+): track 0.00 -> 8.51 mm
- net Net-(IC20-3IN+): track 0.00 -> 8.51 mm
- net Net-(IC5-3IN+): track 0.00 -> 8.51 mm
- net Net-(IC4-3IN+): track 0.00 -> 8.51 mm
- net Net-(IC3-3IN+): track 0.00 -> 8.51 mm
- net Net-(IC22-3IN+): track 0.00 -> 8.51 mm
- net Net-(IC21-3IN+): track 0.00 -> 8.51 mm
- net Net-(IC2-3IN+): track 0.00 -> 8.51 mm
- net Net-(IC20-4IN+): track 0.00 -> 8.44 mm
- net Net-(IC24-4IN+): track 0.00 -> 8.44 mm
- net Net-(IC5-4IN+): track 0.00 -> 8.44 mm
- net Net-(IC4-4IN+): track 0.00 -> 8.44 mm
- net Net-(IC22-4IN+): track 0.00 -> 8.44 mm
- net Net-(IC21-4IN+): track 0.00 -> 8.44 mm
- net Net-(IC3-4IN+): track 0.00 -> 8.44 mm
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Other:
- board size 153.5 x 73.7 mm -> 125 x 90 mm
- board text added: "1"
- board text added: "10"
- board text added: "11"
- board text added: "12"
- board text added: "13"
- board text added: "14"
- board text added: "15"
- board text added: "16"
- board text added: "17"
- board text added: "18"
- board text added: "19"
- board text added: "2"
- board text added: "20"
- board text added: "21"
- board text added: "22"
- board text added: "23"
- board text added: "24"
- board text added: "25"
- board text added: "26"
- board text added: "27"
- board text added: "28"
- board text added: "29"
- board text added: "3"
- board text added: "30"
- board text added: "31"
- board text added: "32"
- board text added: "33"
- board text added: "34"
- board text added: "35"
- board text added: "36"
- board text added: "37"
- board text added: "38"
- board text added: "39"
- board text added: "4"
- board text added: "40"
- board text added: "5"
- board text added: "6"
- board text added: "7"
- board text added: "8"
- board text added: "9"
